File: obd32.kicad_pcb (KiCad board)
At the start: 2 copper layers, 44.2 x 58.7 mm, 69 parts, among them IC1 ATA6561-GAQW-N, IC2 BTS4141N, IC3 LMR14020QDPRTQ1, J1 Conn_01x02_Male, J2 Conn_01x04_Male, J3 Conn_02x05_Odd_Even, J5 OBD2, J9 USB_C_Receptacle_USB2.0, Q1 BC817, Q2 BC817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

Commit message: fix design rule check faults
Parts:
- moved F1 0.51 mm to (207.5, 71.4)
Routing:
- net +BATT: track 4.49 -> 3.98 mm
